Commit message: Dextreme and ADR release

File: assets/urdf/objects/cube_multicolor_allegro_sdf.urdf (robot description, URDF)
Before this commit: robot object, 1 links, 0 joints
Links:
- link object: geometry collision mesh filename=meshes/cube_multicolor.obj scale=.065 .065 .065; visual mesh filename=meshes/cube_multicolor.obj scale=.065 .065 .065

File: assets/urdf/objects/cube_multicolor_dextreme.urdf (robot description, URDF)
Before this commit: robot object, 1 links, 0 joints
Links:
- link object: geometry collision box size=0.065 0.065 0.065; visual mesh filename=meshes/dex_cube.obj scale=.0325 .0325 .0325
