Commit message: 能举起Cube

File: assets/urdf/Lite6SW_/urdf/Lite6SW_.urdf (robot description, URDF)
Before this commit: robot Lite6SW_, 13 links, 12 joints
Links:
- link F1point: geometry collision box size=0.013 0.004 0.013; visual mesh filename=package://Lite6SW_/meshes/F1point.STL
- link F2point: geometry collision box size=0.013 0.004 0.013; visual mesh filename=package://Lite6SW_/meshes/F2point.STL
- link GripSite: geometry visual mesh filename=package://Lite6SW_/meshes/GripSite.STL

File: assets/urdf/Lite6_/urdf/Lite6_.urdf (robot description, URDF)
Before this commit: robot Lite6_, 13 links, 12 joints
Links:
- link F1point: geometry visual mesh filename=package://Lite6_/meshes/F1point.STL
- link F2point: geometry visual mesh filename=package://Lite6_/meshes/F2point.STL
- link GripSite: geometry visual mesh filename=package://Lite6_/meshes/GripSite.STL
