Commit message: 实现Cube堆叠

File: assets/urdf/Lite6SW3/urdf/Lite6SW3.urdf (robot description, URDF)
Before this commit: robot Lite6SW3, 13 links, 12 joints
Joints:
- joint Joint1: limit lower=-3.14 upper=3.14 effort=87 velocity=1 -> lower=-3.14 upper=3.14 effort=187 velocity=1
- joint Joint2: limit lower=-3.14 upper=3.14 effort=87 velocity=1 -> lower=-3.14 upper=3.14 effort=187 velocity=1
- joint Joint3: limit lower=-3.14 upper=3.14 effort=87 velocity=1 -> lower=-3.14 upper=3.14 effort=187 velocity=1
- joint Joint4: limit lower=-3.14 upper=3.14 effort=87 velocity=1 -> lower=-3.14 upper=3.14 effort=187 velocity=1
- joint Joint5: limit lower=-3.14 upper=3.14 effort=12 velocity=1 -> lower=-3.14 upper=3.14 effort=24 velocity=1
- joint Joint6: limit lower=-3.14 upper=3.14 effort=12 velocity=1 -> lower=-3.14 upper=3.14 effort=24 velocity=1
