Commit message: priv obs name to mpc_obs

File: assets/urdf/puck.urdf (robot description, URDF)
Before this commit: robot puck, 1 links, 0 joints
Links:
- link puck: mass 0.5 -> 0.1

Commit message: CoM Randomization

File: assets/urdf/puck.urdf (robot description, URDF)
Before this commit: robot puck, 1 links, 0 joints
Links:
- link puck: geometry collision cylinder length=0.0254 radius=0.0381; visual cylinder length=0.0254 radius=0.0381

Commit message: bigger puck

File: assets/urdf/puck.urdf (robot description, URDF)
Before this commit: robot puck, 1 links, 0 joints
Links:
- link puck: geometry collision cylinder length=0.04 radius=0.055; visual cylinder length=0.04 radius=0.055
