Commit message: stuff

File: assets/urdf/kuka_allegro_description/kuka.urdf (robot description, URDF)
Before this commit: robot kuka_allegro, 10 links, 9 joints
Joints:
- joint iiwa7_joint_7: limit lower=-3.05432619099 upper=3.05432619099 effort=300 velocity=10 -> lower=-6.28319 upper=6.28319 effort=300 velocity=10

File: assets/urdf/kuka_allegro_description/kuka_allegro_touch_sensor.urdf (robot description, URDF)
Before this commit: robot kuka_allegro, 28 links, 27 joints
Joints:
- joint iiwa7_joint_7: limit lower=-3.05432619099 upper=3.05432619099 effort=300 velocity=10 -> lower=-6.28319 upper=6.28319 effort=300 velocity=10

Commit message: fixing hand limits plus rnd

File: assets/urdf/kuka_allegro_description/kuka.urdf (robot description, URDF)
Before this commit: robot kuka_allegro, 10 links, 9 joints
Joints:
- joint iiwa7_joint_7: limit lower=-6.28319 upper=6.28319 effort=300 velocity=10 -> lower=-6.27 upper=6.27 effort=300 velocity=10

File: assets/urdf/kuka_allegro_description/kuka_allegro_touch_sensor.urdf (robot description, URDF)
Before this commit: robot kuka_allegro, 28 links, 27 joints
Joints:
- joint iiwa7_joint_7: limit lower=-6.28319 upper=6.28319 effort=300 velocity=10 -> lower=-6.27 upper=6.27 effort=300 velocity=10
